File: hardware/kicad/esp32_internet_radio_v4/esp32_internet_radio_v4.kicad_pcb (KiCad board)
At the start: 2 copper layers, 68.6 x 53.3 mm, 24 parts, among them J1 ENCODER, J2 RGB LED, J3 ST7789, J4 extend, J5 POWER_IN_5V, J6 PCM5102, J7 TFT_SPI, P1 Power, P2 Analog, P3 Digital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

Commit message: update schematics (pinout)
Connections:
- J1 pad 1: ESPDUINO_IO36 -> ENCODER_CLK
- P2 pad 3: ESPDUINO_IO36 -> ENCODER_CLK
- P2 pad 5: ESPDUINO_IO38 -> ESPDUINO_IO36
- P3 pad 2: ESPDUINO_IO38 -> ESPDUINO_IO36
Routing:
- net ESPDUINO_IO38: track 79.8 -> 0.00 mm, vias 1 -> 0
- net ENCODER_CLK: track 0.00 -> 46.6 mm, vias 0 -> 1
- net ESPDUINO_IO36: track 46.6 -> 79.8 mm
Changed lines of the file:
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@@
   (net 8 "/AREF")
   (net 9 "ESPDUINO_IO34")
-  (net 10 "ESPDUINO_IO38")
+  (net 10 "ENCODER_CLK")
   (net 11 "ESPDUINO_IO15")
   (net 12 "unconnected-(P5-Pad1)")
@@
       (net 7 "ESPDUINO_IO4") (pinfunction "Pin_2") (pintype "passive"))
     (pad "3" thru_hole oval locked (at 5.08 0) (size 1.7272 2.032) (drill 1.016) (layers *.Cu *.Mask "F.SilkS")
-      (net 39 "ESPDUINO_IO36") (pinfunction "Pin_3") (pintype "passive"))
+      (net 10 "ENCODER_CLK") (pinfunction "Pin_3") (pintype "passive"))
     (pad "4" thru_hole oval locked (at 7.62 0) (size 1.7272 2.032) (drill 1.016) (layers *.Cu *.Mask "F.SilkS")
       (net 9 "ESPDUINO_IO34") (pinfunction "Pin_4") (pintype "passive"))
     (pad "5" thru_hole oval locked (at 10.16 0) (size 1.7272 2.032) (drill 1.016) (layers *.Cu *.Mask "F.SilkS")
-      (net 10 "ESPDUINO_IO38") (pinfunction "Pin_5") (pintype "passive+no_connect"))
+      (net 39 "ESPDUINO_IO36") (pinfunction "Pin_5") (pintype "passive+no_connect"))
     (pad "6" thru_hole oval locked (at 12.7 0) (size 1.7272 2.032) (drill 1.016) (layers *.Cu *.Mask "F.SilkS")
       (net 3 "ENCODER_DT") (pinfunction "Pin_6") (pintype "passive"))
@@
       (net 3 "ENCODER_DT") (pinfunction "Pin_1") (pintype "passive"))
     (pad "2" thru_hole oval locked (at 2.54 0) (size 1.7272 2.032) (drill 1.016) (layers *.Cu *.Mask "F.SilkS")
-      (net 10 "ESPDUINO_IO38") (pinfunction "Pin_2") (pintype "passive+no_connect"))
+      (net 39 "ESPDUINO_IO36") (pinfunction "Pin_2") (pintype "passive+no_connect"))
     (pad "3" thru_hole oval locked (at 5.08 0) (size 1.7272 2.032) (drill 1.016) (layers *.Cu *.Mask "F.SilkS")
       (net 8 "/AREF") (pinfunction "Pin_3") (pintype "passive+no_connect"))
@@
     (fp_line (start -1.52 7.92) (end 0 7.92) (layer "F.Fab") (width 0.1))
     (pad "1" thru_hole rect (at 0 0 180) (size 1.7 1.7) (drill 1) (layers *.Cu *.Mask)
-      (net 39 "ESPDUINO_IO36") (pinfunction "Pin_1") (pintype "passive"))
+      (net 10 "ENCODER_CLK") (pinfunction "Pin_1") (pintype "passive"))
     (pad "2" thru_hole oval (at 0 2.54 180) (size 1.7 1.7) (drill 1) (layers *.Cu *.Mask)
       (net 3 "ENCODER_DT") (pinfunction "Pin_2") (pintype "passive"))
@@
   (segment (start 150.1631 83.4168) (end 152.4204 81.1595) (width 0.5) (layer "B.Cu") (net 7))
   (segment (start 164.338 123.825) (end 162.8529 125.3101) (width 0.5) (layer "B.Cu") (net 7))
-  (segment (start 171.958 123.825) (end 158.3859 110.2529) (width 0.5) (layer "F.Cu") (net 10))
-  (segment (start 158.3859 110.2529) (end 135.7975 110.2529) (width 0.5) (layer "F.Cu") (net 10))
-  (via (at 135.7975 110.2529) (size 0.6) (drill 0.4) (layers "F.Cu" "B.Cu") (net 10))
-  (segment (start 135.7974 110.2529) (end 135.7975 110.2529) (width 0.5) (layer "B.Cu") (net 10))
-  (segment (start 129.9987 85.1328) (end 135.7974 90.9315) (width 0.5) (layer "B.Cu") (net 10))
-  (segment (start 129.9987 77.9003) (end 129.9987 85.1328) (width 0.5) (layer "B.Cu") (net 10))
-  (segment (start 135.7974 90.9315) (end 135.7974 110.2529) (width 0.5) (layer "B.Cu") (net 10))
-  (segment (start 132.334 75.565) (end 129.9987 77.9003) (width 0.5) (layer "B.Cu") (net 10))
+  (segment (start 166.878 123.825) (end 165.1176 122.0646) (width 0.5) (layer "F.Cu") (net 10))
+  (segment (start 165.1176 122.0646) (end 142.8197 122.0646) (width 0.5) (layer "F.Cu") (net 10))
+  (via (at 142.8197 122.0646) (size 0.6) (drill 0.4) (layers "F.Cu" "B.Cu") (net 10))
+  (segment (start 131.838 104.77) (end 131.838 111.0829) (width 0.5) (layer "B.Cu") (net 10))
+  (segment (start 131.838 111.0829) (end 142.8197 122.0646) (width 0.5) (layer "B.Cu") (net 10))
   (segment (start 162.7147 77.1883) (end 152.2882 77.1883) (width 0.5) (layer "F.Cu") (net 16))
   (segment (start 164.338 75.565) (end 162.7147 77.1883) (width 0.5) (layer "F.Cu") (net 16))
@@
   (segment (start 135.0593 100.3713) (end 131.838 97.15) (width 0.5) (layer "B.Cu") (net 35))
   (segment (start 173.6776 85.3157) (end 172.0158 85.3157) (width 0.5) (layer "B.Cu") (net 35))
-  (segment (start 166.878 123.825) (end 165.1176 122.0646) (width 0.5) (layer "F.Cu") (net 39))
-  (segment (start 165.1176 122.0646) (end 142.8197 122.0646) (width 0.5) (layer "F.Cu") (net 39))
-  (via (at 142.8197 122.0646) (size 0.6) (drill 0.4) (layers "F.Cu" "B.Cu") (net 39))
-  (segment (start 131.838 104.77) (end 131.838 111.0829) (width 0.5) (layer "B.Cu") (net 39))
-  (segment (start 131.838 111.0829) (end 142.8197 122.0646) (width 0.5) (layer "B.Cu") (net 39))
+  (segment (start 171.958 123.825) (end 158.3859 110.2529) (width 0.5) (layer "F.Cu") (net 39))
+  (segment (start 158.3859 110.2529) (end 135.7975 110.2529) (width 0.5) (layer "F.Cu") (net 39))
+  (via (at 135.7975 110.2529) (size 0.6) (drill 0.4) (layers "F.Cu" "B.Cu") (net 39))
+  (segment (start 135.7974 110.2529) (end 135.7975 110.2529) (width 0.5) (layer "B.Cu") (net 39))
+  (segment (start 129.9987 85.1328) (end 135.7974 90.9315) (width 0.5) (layer "B.Cu") (net 39))
+  (segment (start 129.9987 77.9003) (end 129.9987 85.1328) (width 0.5) (layer "B.Cu") (net 39))
+  (segment (start 135.7974 90.9315) (end 135.7974 110.2529) (width 0.5) (layer "B.Cu") (net 39))
+  (segment (start 132.334 75.565) (end 129.9987 77.9003) (width 0.5) (layer "B.Cu") (net 39))
   (zone (net 17) (net_name "ENCODER_GND") (layers F&B.Cu) (hatch edge 0.508)
     (connect_pads (clearance 0.508))

Commit message: updated schematics and pcb
Parts:
- J1: footprint Connector_PinSocket_2.54mm:PinSocket_1x05_P2.54mm_Horizontal -> Connector_PinHeader_2.54mm:PinHeader_1x05_P2.54mm_Vertical
- moved J6 6.38 mm to (126.2, 109.9)
- moved kibuzzard-6279C2C8 3.81 mm to (119.9, 116.2)
Connections:
- P3 pad 1: ENCODER_DT -> unconnected-(P3-Pad1)
- P3 pad 2: ESPDUINO_IO36 -> unconnected-(P3-Pad2)
Routing:
- net ESPDUINO_IO36: track 79.8 -> 0.00 mm, vias 1 -> 0
- net ENCODER_DT: track 80.2 -> 51.6 mm, vias 1 -> 0
- net ESPDUINO_IO4: track 68.7 -> 41.7 mm
- net ESPDUINO_3.3V: track 137.2 -> 117.8 mm, vias 1 -> 0
- net ESPDUINO_IO2: track 59.4 -> 41.7 mm
- net ESPDUINO_IO23: track 33.4 -> 19.9 mm, vias 1 -> 0
- net ESPDUINO_IO27: track 63.3 -> 54.7 mm
- net ESPDUINO_IO5: track 49.5 -> 41.2 mm
- net ESPDUINO_IO14: track 44.5 -> 36.5 mm, vias 0 -> 1
- net ESPDUINO_IO16: track 44.5 -> 38.7 mm
- net ESPDUINO_IO25: track 70.2 -> 66.6 mm
- net ENCODER_CLK: track 46.6 -> 43.2 mm, vias 1 -> 0
- net ESPDUINO_IO13: track 34.7 -> 38.0 mm, vias 2 -> 1
- net ESPDUINO_IO26: track 70.5 -> 67.3 mm, vias 0 -> 1
- net ESPDUINO_IO18: track 25.5 -> 22.5 mm, vias 1 -> 0
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
Commit message: update silk
Parts:
- moved kibuzzard-6279C2C8 10.2 mm to (119.9, 106.0)
- moved kibuzzard-6279C2B7 9.41 mm to (135.1, 99.7)
Changed lines of the file:
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@@
     (property "Sheetname" "")
     (attr through_hole)
-    (fp_text reference "P3" (at 11.43 2.794) (layer "F.SilkS")
+    (fp_text reference "P3" (at 11.43 2.794) (layer "F.SilkS") hide
       (effects (font (size 1 1) (thickness 0.15)))
     )
@@
   )
   (footprint "kibuzzard-6279C2C8" (layer "F.Cu")
-    (at 119.888 116.205)
+    (at 119.888 106.045)
     (descr "Converted using: scripting")
     (tags "svg2mod")
@@
   )
   (footprint "kibuzzard-6279C2B7" (layer "F.Cu")
-    (at 144.538 99.695 -90)
+    (at 135.128 99.695 -90)
     (descr "Converted using: scripting")
     (tags "svg2mod")
@@
   (gr_line (start 175.514 73.025) (end 110.998 73.025) (layer "Edge.Cuts") (width 0.15))
   (gr_line (start 177.038 85.979) (end 177.038 74.549) (layer "Edge.Cuts") (width 0.15))
-  (gr_text "LCK" (at 118.618 113.665 90) (layer "F.SilkS")
+  (gr_text "LCK" (at 118.618 114.935 90) (layer "F.SilkS")
     (effects (font (size 1 1) (thickness 0.15)) (justify left))
   )
@@
     (effects (font (size 1 1) (thickness 0.15)) (justify left))
   )
-  (gr_text "3V3" (at 113.538 113.665 90) (layer "F.SilkS")
-    (effects (font (size 1 1) (thickness 0.15)) (justify left))
-  )
-  (gr_text "BCK" (at 123.698 113.665 90) (layer "F.SilkS")
+  (gr_text "3V3" (at 113.538 114.935 90) (layer "F.SilkS")
+    (effects (font (size 1 1) (thickness 0.15)) (justify left))
+  )
+  (gr_text "BCK" (at 123.698 114.935 90) (layer "F.SilkS")
     (effects (font (size 1 1) (thickness 0.15)) (justify left))
   )
@@
     (effects (font (size 1 1) (thickness 0.15)) (justify left))
   )
-  (gr_text "SCK" (at 126.238 113.665 90) (layer "F.SilkS")
+  (gr_text "SCK" (at 126.238 114.935 90) (layer "F.SilkS")
     (effects (font (size 1 1) (thickness 0.15)) (justify left))
   )
@@
     (effects (font (size 1 1) (thickness 0.15)) (justify left))
   )
-  (gr_text "GND" (at 116.078 113.665 90) (layer "F.SilkS")
+  (gr_text "GND" (at 116.078 114.935 90) (layer "F.SilkS")
     (effects (font (size 1 1) (thickness 0.15)) (justify left))
   )
@@
     (effects (font (size 1 1) (thickness 0.15)) (justify left))
   )
-  (gr_text "DIN" (at 121.158 113.665 90) (layer "F.SilkS")
-    (effects (font (size 1 1) (thickness 0.15)) (justify left))
-  )
+  (gr_text "DIN" (at 121.158 114.935 90) (layer "F.SilkS")
+    (effects (font (size 1 1) (thickness 0.15)) (justify left))
+  )
